Commit message: Added inertial tags

File: src/helios/urdfs/helios.urdf (robot description, URDF)
Before this commit: robot helios, 3 links, 10 joints
Links:
- link base_link: mass None -> 0.1
- link camera_link: mass None -> 0.015
- link lidar_link: mass None -> 0.04

File: src/helios/urdfs/helios.xacro (robot description, xacro)
@@ -1,4 +1,5 @@
 <?xml version="1.0"?>
 <robot xmlns:xacro="http://www.ros.org/wiki/xacro">
+    <!-- Colors-->
     <material name="red">
         <color rgba="1.0 0.0 0.0 1.0"/>
@@ -16,4 +17,18 @@
         <color rgba="1.0 1.0 1.0 1.0"/>
     </material>
+    <!-- Properties-->
+    <xacro:property name="propeller_mass" value="0.05"/>
+    <xacro:property name="propeller_rad" value="0.02"/>
+    <xacro:property name="propeller_ht" value="0.01"/>
+    <xacro:property name="stand_mass" value="0.02"/>
+    <xacro:property name="stand_rad" value="0.01"/>
+    <xacro:property name="stand_ht" value="0.05"/>
+    <!-- Macros-->
+    <xacro:macro name="cyl_inertia" params="mass rad ht">
+        <inertia ixx="{(mass/12)*(3*rad*rad+ht*ht)}" ixy="0.0" ixz="0.0" iyy="{(mass/12)*(3*rad*rad+ht*ht)}" iyz="0.0" izz="{(mass/2)*(rad*rad)}"/>
+    </xacro:macro>
+    <xacro:macro name="box_inertia" params="mass w d h">
+        <inertia ixx="{(mass/12)*(h*h+d*d)}" ixy="0.0" ixz="0.0" iyy="{(mass/12)*(w*w+h*h)}" iyz="0.0" izz="{(mass/12)*(w*w+d*d)}"/>
+    </xacro:macro>
     <xacro:macro name="propeller_link" params="pref suff">
         <link name="${pref}_propeller_${suff}">
@@ -26,8 +41,14 @@
             </visual>
             <collision>
+                <origin xyz="0.0 0.0 0.0" rpy="0.0 0.0 0.0"/>
                 <geometry>
                     <cylinder radius="0.02" length="0.01"/>
                 </geometry>
             </collision>
+            <inertial>
+                <origin xyz="0.0 0.0 0.0" rpy="0.0 0.0 0.0"/>
+                <mass value="${propeller_mass}"/>
+                <xacro:cyl_inertia mass="{propeller_mass}" rad="{propeller_rad}" ht="{propeller_ht}"/>
+            </inertial>
         </link>
     </xacro:macro>
@@ -42,8 +63,14 @@
             </visual>
             <collision>
+                <origin xyz="0.0 0.0 0.0" rpy="0.0 0.0 0.0"/>
                 <geometry>
                     <cylinder radius="0.01" length="0.05"/>
                 </geometry>
             </collision>
+            <inertial>
+                <origin xyz="0.0 0.0 0.0" rpy="0.0 0.0 0.0"/>
+                <mass value="${stand_mass}"/>
+                <xacro:cyl_inertia mass="{stand_mass}" rad="{stand_rad}" ht="{stand_ht}"/>
+            </inertial>
         </link>
     </xacro:macro>
