Commit message: Added xacro files and gazebo launch file

File: src/helios/urdfs/helios_main.urdf.xacro (robot description, xacro)
@@ -1,5 +1,12 @@
 <?xml version="1.0"?>
 <robot xmlns:xacro="http://www.ros.org/wiki/xacro" name="helios">
-    <xacro:include filename="helios.xacro"/>
+    <xacro:include filename="helios.urdf.xacro"/>
+    <!-- Dummy Link and Dummy Joint -->
+    <link name="dummy_link" />
+    <joint name="base_to_dummy" type="fixed">
+    <parent link="dummy_link" />
+    <child link="base_link" />
+    </joint>
+    <!-- Base Link -->
     <link name="base_link">
         <visual>
@@ -7,5 +14,5 @@
                 <box size="0.2 0.2 0.05"/>
             </geometry>
-            <origin xyz="0.0 0.0 0.075" rpy="0.0 0.0 0.0"/>
+            <origin xyz="0 0 0.075" rpy="0 0 0"/>
             <material name="black"/>
         </visual>
@@ -14,11 +21,7 @@
                 <box size="0.2 0.2 0.05"/>
             </geometry>
-            <origin xyz="0.0 0.0 0.075" rpy="0.0 0.0 0.0"/>
+            <origin xyz="0 0 0.075" rpy="0 0 0"/>
         </collision>
-        <inertial>
-            <origin xyz="0.0 0.0 0.075" rpy="0.0 0.0 0.0"/>
-            <mass value="0.1"/>
-            <xacro:box_inertia mass="0.1" w="0.2" d="0.2" h="0.05"/>
-        </inertial>
+        <xacro:box_inertia mass="0.1" w="0.2" d="0.2" h="0.05"/>
     </link>
     <!-- Propeller links -->
@@ -93,9 +96,5 @@
             </geometry>
         </collision>
-        <inertial>
-            <origin xyz="0.0 0.0 0.0" rpy="0.0 0.0 0.0"/>
-            <mass value="0.015"/>
-            <xacro:box_inertia mass="0.015" w="0.04" d="0.04" h="0.04"/>
-        </inertial>
+        <xacro:box_inertia mass="0.015" w="0.04" d="0.04" h="0.04"/>
     </link>
     <link name="lidar_link">
@@ -113,9 +112,5 @@
             </geometry>
         </collision>
-        <inertial>
-            <origin xyz="0.0 0.0 0.0" rpy="0.0 0.0 0.0"/>
-            <mass value="0.04"/>
-            <xacro:box_inertia mass="0.04" w="0.03" d="0.03" h="0.03"/>
-        </inertial>
+        <xacro:box_inertia mass="0.04" w="0.03" d="0.03" h="0.03"/>
     </link>
     <!-- Sensor Joints-->
@@ -132,46 +127,56 @@
     <!-- Gazebo Sensor Plugins -->
     <gazebo reference="camera_link">
-        <sensor type="camera" name="camera_sensor">
+        <plugin
+          filename="libignition-gazebo-sensors-system.so"
+          name="ignition::gazebo::systems::Sensors">
+          <sensor name="camera_sensor" type="camera">
+            <always_on>1</always_on>
             <update_rate>30</update_rate>
+            <topic>/camera/image_raw</topic>
             <camera>
-                <horizontal_fov>1.047</horizontal_fov>
-                <image>
-                    <width>640</width>
-                    <height>480</height>
-                    <format>R8G8B8</format>
-                </image>
-                <clip>
-                    <near>0.1</near>
-                    <far>100</far>
-                </clip>
+              <horizontal_fov>1.047</horizontal_fov>
+              <image>
+                <width>640</width>
+                <height>480</height>
+                <format>R8G8B8</format>
+              </image>
+              <clip>
+                <near>0.1</near>
+                <far>100.0</far>
+              </clip>
             </camera>
-            <plugin name="gazebo_ros_camera" filename="libgazebo_ros_camera.so"/>
-        </sensor>
+          </sensor>
+        </plugin>
     </gazebo>
     <gazebo reference="lidar_link">
-        <sensor type="gpu_ray" name="lidar_sensor">
+        <plugin
+          filename="libignition-gazebo-sensors-system.so"
+          name="ignition::gazebo::systems::Sensors">
+          <sensor name="lidar_sensor" type="gpu_ray">
+            <always_on>1</always_on>
             <update_rate>10</update_rate>
+            <topic>/lidar/scan</topic>
             <ray>
-                <scan>
-                    <horizontal>
-                        <samples>720</samples>
-                        <resolution>1</resolution>
-                        <min_angle>-1.57</min_angle>
-                        <max_angle>1.57</max_angle>
-                    </horizontal>
-                    <vertical>
-                        <samples>1</samples>
-                        <min_angle>0</min_angle>
-                        <max_angle>0</max_angle>
-                    </vertical>
-                </scan>
-                <range>
-                    <min>0.2</min>
-                    <max>30.0</max>
-                    <resolution>0.01</resolution>
-                </range>
+              <scan>
+                <horizontal>
+                  <samples>720</samples>
+                  <resolution>1</resolution>
+                  <min_angle>-1.57</min_angle>
+                  <max_angle>1.57</max_angle>
+                </horizontal>
+                <vertical>
+                  <samples>1</samples>
+                  <min_angle>0</min_angle>
+                  <max_angle>0</max_angle>
+                </vertical>
+              </scan>
+              <range>
+                <min>0.2</min>
+                <max>30.0</max>
+                <resolution>0.01</resolution>
+              </range>
             </ray>
-            <plugin name="gazebo_ros_laser" filename="libgazebo_ros_gpu_laser.so"/>
-        </sensor>
+          </sensor>
+        </plugin>
     </gazebo>
 </robot>

Commit message: Added TF Publisher, Changed HELIOS Models.

File: src/helios/urdfs/helios_main.urdf.xacro (robot description, xacro)
@@ -118,5 +118,5 @@
         <parent link="base_link"/>
         <child link="camera_link"/>
-        <origin xyz="0.0 0.0 0.025" rpy="0.0 0.0 0.0"/>
+        <origin xyz="0.0 0.0 0.030" rpy="0.0 0.0 0.0"/>
     </joint>
     <joint name="lidar_joint" type="fixed">
